File: pcb/prrplsattiny20.kicad_sch (KiCad schematic)
At the start: 23 parts, among them J1 Conn_02x08_Counter_Clockwise, J2 SEI-105-02-GF-S-M-AT, U1 ATtiny20-UUR

Commit message: checkpoint
Connections:
- net B: no longer D2.1 (K), D5.2 (A), D6.1 (K), D7.2 (A)
- net A renamed PA6
- net C renamed PA5
- new net PB2: D2.1 (K), D5.2 (A), D6.1 (K), D7.2 (A)
Changed lines of the file:
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@@
 		)
 	)
-	(label "B"
+	(label "PB2"
 		(at 182.88 90.17 0)
 		(effects
@@
 		)
 	)
-	(label "C"
+	(label "PA5"
 		(at 203.2 106.68 0)
 		(effects
@@
 		)
 	)
-	(label "C"
+	(label "PA5"
 		(at 165.1 114.3 0)
 		(effects
@@
 		)
 	)
-	(label "A"
+	(label "PA6"
 		(at 165.1 116.84 0)
 		(effects
@@
 		)
 	)
-	(label "A"
+	(label "PA6"
 		(at 193.04 105.41 0)
 		(effects
