File: pcb/prrplsattiny20.kicad_sch (KiCad schematic)
At the start: 23 parts, among them J1 Conn_02x08_Counter_Clockwise, J2 SEI-105-02-GF-S-M-AT, U1 ATtiny20-UUR

Commit message: v2 of the pcb
Parts:
- removed FID1: Fiducial, Fiducial:Fiducial_0.5mm_Mask1mm, symbol Mechanical:Fiducial
- removed J2: SEI-105-02-GF-S-M-AT, JSK:sei-105-mating, symbol SEI-105-02-GF-S-M-AT:SEI-105-02-GF-S-M-AT
- removed JP1001, JP1002, JP1003, JP1004, JP1005: SolderJumper_2_Open, JSK:solderbridge_R_0201_0603Metric_as_solderbridge, symbol Jumper:SolderJumper_2_Open
- removed TP1001, TP1002, TP1003, TP1004, TP1005: TestPoint, JSK:TestPoint_Keystone_1005, symbol Connector:TestPoint
- added C1001: 22μF, Capacitor_SMD:C_0402_1005Metric, symbol Device:C
- added D1001, D1002, D1003, D1004, D1005, D1006: YELLOW LED, LED_SMD:LED_0402_1005Metric, symbol Device:LED
- added J1001, J1002, J1003, J1004, J1005, J1006: Conn_01x01, JSK:SolderWire-D0.7mm_Drill0.3, symbol Connector_Generic:Conn_01x01
- J1: footprint JSK:16-pin-clip-dbg -> Connector:Tag-Connect_TC2030-IDC-NL_2x03_P1.27mm_Vertical; symbol Connector_Generic:Conn_02x08_Counter_Clockwise -> Connector_Generic:Conn_02x03_Odd_Even; now in the parts list
Connections:
- net +5V: now also C1001.1, J1002.1 (Pin_1), J1004.1 (Pin_1)
- net GND: now also D1.1 (K), D2.1 (K), D3.1 (K), D5.1 (K), D6.1 (K), D7.1 (K), J1.6 (Pin_6), C1001.2, J1005.1 (Pin_1), J1006.1 (Pin_1); no longer J1.1 (Pin_1), U1.A3 (PA1)
- net PA5: now also D1003.1 (K), D1004.2 (A), D1005.2 (A), D1006.1 (K); no longer D1.1 (K), D3.2 (A), D6.2 (A), D7.1 (K), U1.C1 (PA5)
- net PA6: now also D1001.2 (A), D1002.1 (K), D1003.2 (A), D1004.1 (K); no longer D1.2 (A), D2.2 (A), D3.1 (K), D5.1 (K), U1.B2 (PA6)
- net PB2: now also D1001.1 (K), D1002.2 (A), D1005.1 (K), D1006.2 (A); no longer D2.1 (K), D5.2 (A), D6.1 (K), D7.2 (A)
- net TPIDATA: now also D7.2 (A), J1.1 (Pin_1); no longer J1.4 (Pin_4)
- net A5: now reaches U1.A5 (PA2)
- net A5: now also D5.2 (A)
- net Serial_In: now reaches U1.C3 (PA7)
- net Serial_In: now also J1.4 (Pin_4), J1003.1 (Pin_1)
- net B renamed D2
- net D2: now also D6.2 (A)
- net CENTER renamed A1
- net TPICLK renamed TPICLK_SO
- net TPICLK_SO: now also J1001.1 (Pin_1)
- new net A3: D2.2 (A), U1.A3 (PA1)
- new net B2: D1.2 (A), U1.B2 (PA6)
- new net C1: D3.2 (A), U1.C1 (PA5)
