File: pcb/prrplsattiny20.kicad_pcb (KiCad board)
At the start: 4 copper layers, 18 x 13.9 mm, 22 parts, among them J1 Conn_02x08_Counter_Clockwise, J2 SEI-105-02-GF-S-M-AT, U1 ATtiny20-UUR

Commit message: checkpoint
Parts:
- added FID1: Fiducial, Fiducial:Fiducial_0.5mm_Mask1mm, F.Cu at (0.78, 0.78)
Connections:
- net /A renamed /PA6
- net /C renamed /PA5
- D2 pad 1: /B -> /PB2
- D5 pad 2: /B -> /PB2
- D6 pad 1: /B -> /PB2
- D7 pad 2: /B -> /PB2

Commit message: v2 of the pcb
Parts:
- removed FID1: Fiducial, Fiducial:Fiducial_0.5mm_Mask1mm
- removed J2: SEI-105-02-GF-S-M-AT, JSK:sei-105-mating
- removed JP1001, JP1002, JP1003, JP1004, JP1005: SolderJumper_2_Open, JSK:solderbridge_R_0201_0603Metric_as_solderbridge
- removed TP1001, TP1002, TP1003, TP1004, TP1005: TestPoint, JSK:TestPoint_Keystone_1005
- added C1001: 22μF, Capacitor_SMD:C_0402_1005Metric, F.Cu at (141.8, 72.8)
- added J1001: Conn_01x01, JSK:SolderWire-D0.7mm_Drill0.3, F.Cu at (136.8, 70.8)
- added J1002: Conn_01x01, JSK:SolderWire-D0.7mm_Drill0.3, F.Cu at (140.5, 69.7)
- added J1003: Conn_01x01, JSK:SolderWire-D0.7mm_Drill0.3, F.Cu at (141.9, 71.2)
- added J1004: Conn_01x01, JSK:SolderWire-D0.7mm_Drill0.3, F.Cu at (137.9, 69.4)
- added J1005: Conn_01x01, JSK:SolderWire-D0.7mm_Drill0.3, F.Cu at (141.3, 70.5)
- added J1006: Conn_01x01, JSK:SolderWire-D0.7mm_Drill0.3, F.Cu at (137.3, 70.1)
- J1: footprint JSK:16-pin-clip-dbg -> Connector:Tag-Connect_TC2030-IDC-NL_2x03_P1.27mm_Vertical; moved to B.Cu
- moved J1 11.0 mm to (140.1, 72.7), turned to 135 degrees
- moved R1 0.75 mm to (140.3, 70.8), turned to 135 degrees
- moved C1 0.48 mm to (140.4, 73.8)
Connections:
- net /CENTER renamed /A1
- net /TPICLK renamed /TPICLK_SO
- D1 pad 1: /PA5 -> GND
- D1 pad 2: /PA6 -> /B2
- D2 pad 1: /PB2 -> GND
- D2 pad 2: /PA6 -> /A3
- D3 pad 1: /PA6 -> GND
- D3 pad 2: /PA5 -> /C1
- D5 pad 1: /PA6 -> GND
- D5 pad 2: /PB2 -> /A5
- D6 pad 1: /PB2 -> GND
- D6 pad 2: /PA5 -> /D2
- D7 pad 1: /PA5 -> GND
- D7 pad 2: /PB2 -> /TPIDATA
- J1 pad 1: GND -> /TPIDATA
- J1 pad 4: /TPIDATA -> /Serial_In
- J1 pad 6: unconnected-(J1-Pin_6-Pad6) -> GND
- U1 pad A3: GND -> /A3
- U1 pad A5: unconnected-(U1-PA2-PadA5) -> /A5
- U1 pad B2: /PA6 -> /B2
- U1 pad C1: /PA5 -> /C1
- U1 pad C3: unconnected-(U1-PA7-PadC3) -> /Serial_In
- U1 pad D2: /B -> /D2
Routing:
- net /TPIDATA: track 34.2 -> 3.57 mm, vias 2 -> 1
- net /TPICLK_SO: track 38.4 -> 9.63 mm, vias 2 -> 1
- net /~{RESET}: track 36.9 -> 8.74 mm
- net /PA6: track 18.5 -> 0.00 mm, vias 3 -> 0
- net /PA5: track 15.3 -> 0.00 mm, vias 3 -> 0
- net /B: track 11.3 -> 0.00 mm
- net GND: track 11.1 -> 3.32 mm, vias 3 -> 9
- net /Serial_In: track 0.00 -> 6.26 mm, vias 0 -> 1
- net /B2: track 0.00 -> 6.23 mm
- net /A3: track 0.00 -> 5.49 mm
- net /A5: track 0.00 -> 4.28 mm
- net /C1: track 0.00 -> 2.73 mm
- net +5V: track 14.7 -> 12.8 mm, vias 3 -> 1
- net /D2: track 0.00 -> 1.37 mm
- added copper zone on In1.Cu, net GND
- removed copper zone on In1.Cu, net +5V
Other:
- board size 18 x 13.9 mm -> 8.2 x 8.2 mm
- board text added: "G"
- board text added: "SI"
- board text added: "SO"
- board text added: "SOTC"
- board text added: "TD"
- board text added: "V"
- board text added: "V3.2"
- board text added: "WayWayWay 2542"
- board text added: "~{R}"
- board text removed: "JSK PRR PLS v3.1 2528 WayWayWay"
- board text removed: "⏚ + C D ~{R}"
- board text removed: "⏚+CD~{R}"
