File: pcb/prrplsattiny20_cover.kicad_pcb (KiCad board)
At the start: 4 copper layers, 0 parts

Commit message: v2 of the pcb
Other:
- board outline added: 8 x 8 mm
Changed lines of the file:
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@@
 	)
 	(net 0 "")
+	(gr_circle
+		(center 130.490155 80.060231)
+		(end 130.922383 80.060231)
+		(stroke
+			(width 0.05)
+			(type solid)
+		)
+		(fill no)
+		(layer "Edge.Cuts")
+	)
+	(gr_circle
+		(center 127.1111 76.640713)
+		(end 127.543328 76.640713)
+		(stroke
+			(width 0.05)
+			(type solid)
+		)
+		(fill no)
+		(layer "Edge.Cuts")
+	)
+	(gr_circle
+		(center 130.481848 73.331481)
+		(end 130.914076 73.331481)
+		(stroke
+			(width 0.05)
+			(type solid)
+		)
+		(fill no)
+		(layer "Edge.Cuts")
+	)
+	(gr_circle
+		(center 132.838036 74.307279)
+		(end 133.270264 74.307279)
+		(stroke
+			(width 0.05)
+			(type solid)
+		)
+		(fill no)
+		(layer "Edge.Cuts")
+	)
+	(gr_circle
+		(center 130.45 76.66)
+		(end 134.45 76.66)
+		(stroke
+			(width 0.05)
+			(type solid)
+		)
+		(fill no)
+		(layer "Edge.Cuts")
+	)
+	(gr_circle
+		(center 133.810544 76.642304)
+		(end 134.242772 76.642304)
+		(stroke
+			(width 0.05)
+			(type solid)
+		)
+		(fill no)
+		(layer "Edge.Cuts")
+	)
+	(gr_circle
+		(center 128.107154 79.077093)
+		(end 128.539382 79.077093)
+		(stroke
+			(width 0.05)
+			(type solid)
+		)
+		(fill no)
+		(layer "Edge.Cuts")
+	)
 	(embedded_fonts no)
 )
