File: testcircuit/testcircuit/testcircuit.kicad_sch (KiCad schematic)
At the start: 6 parts, among them J1001 Programming Socket, J1002 Testing Position 2 Socket, J1003 Testing Position 1 Socket, U1001 FT232RL

Commit message: show not-connected in test circuit
Parts:
- added JP1001, JP1002: SolderJumper_2_Open, symbol Jumper:SolderJumper_2_Open
Connections:
- net RX: now also JP1001.1 (A), JP1002.1 (A); no longer A1001.D12 (D12_MISO), A1001.D13 (D13_SCK), J1001.3 (Pin_3), J1001.4 (Pin_4), R1001.2
- new net TPI_CLK: A1001.D13 (D13_SCK), J1001.3 (Pin_3), JP1001.2 (B)
- new net TPI_DATA: A1001.D12 (D12_MISO), J1001.4 (Pin_4), JP1002.2 (B), R1001.2
Changed lines of the file:
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@@
+	)
+	(junction
+		(at 99.06 66.04)
+		(diameter 0)
+		(color 0 0 0 0)
+	)
+	(junction
+		(at 96.52 116.84)
+		(diameter 0)
+		(color 0 0 0 0)
+	)
+	(junction
+		(at 101.6 116.84)
+		(diameter 0)
+		(color 0 0 0 0)
+	)
+	(junction
+		(at 193.04 86.36)
+		(diameter 0)
+		(color 0 0 0 0)
+	)
+	(junction
+		(at 180.34 82.55)
+		(diameter 0)
+		(color 0 0 0 0)
+	)
+	(junction
+		(at 99.06 116.84)
+		(diameter 0)
+		(color 0 0 0 0)
+	)
+	(junction
+		(at 121.92 113.03)
+		(diameter 0)
+		(color 0 0 0 0)
 	)
 	(junction
@@
 	)
 	(junction
-		(at 99.06 66.04)
-		(diameter 0)
-		(color 0 0 0 0)
-	)
-	(junction
-		(at 96.52 116.84)
-		(diameter 0)
-		(color 0 0 0 0)
-	)
-	(junction
-		(at 180.34 82.55)
-		(diameter 0)
-		(color 0 0 0 0)
-	)
-	(junction
-		(at 101.6 116.84)
-		(diameter 0)
-		(color 0 0 0 0)
-	)
-	(junction
-		(at 193.04 86.36)
-		(diameter 0)
-		(color 0 0 0 0)
-	)
-	(junction
-		(at 99.06 116.84)
-		(diameter 0)
-		(color 0 0 0 0)
-	)
-	(junction
-		(at 121.92 113.03)
-		(diameter 0)
-		(color 0 0 0 0)
-	)
-	(junction
 		(at 127 105.41)
 		(diameter 0)
@@
 	(wire
 		(pts
-			(xy 193.04 80.01) (xy 181.61 80.01)
-		)
-		(stroke
-			(width 0)
-			(type default)
-		)
-	)
-	(wire
-		(pts
-			(xy 191.77 82.55) (xy 180.34 82.55)
+			(xy 181.61 69.85) (xy 181.61 80.01)
 		)
 		(stroke
@@
 	(wire
 		(pts
+			(xy 180.34 82.55) (xy 181.61 82.55)
+		)
+		(stroke
+			(width 0)
+			(type default)
+		)
+	)
+	(wire
+		(pts
 			(xy 193.04 54.61) (xy 186.69 54.61)
 		)
@@
 	(wire
 		(pts
-			(xy 181.61 80.01) (xy 181.61 69.85)
-		)
-		(stroke
-			(width 0)
-			(type default)
-		)
-	)
-	(wire
-		(pts
 			(xy 184.15 52.07) (xy 193.04 52.07)
 		)
@@
 	(wire
 		(pts
+			(xy 189.23 82.55) (xy 191.77 82.55)
+		)
+		(stroke
+			(width 0)
+			(type default)
+		)
+	)
+	(wire
+		(pts
 			(xy 193.04 86.36) (xy 200.66 86.36)
 		)
@@
 		(pts
 			(xy 190.5 85.09) (xy 190.5 91.44)
+		)
+		(stroke
+			(width 0)
+			(type default)
+		)
+	)
+	(wire
+		(pts
+			(xy 189.23 80.01) (xy 193.04 80.01)
 		)
 		(stroke
@@
 	)
 	(symbol
+		(lib_name "Conn_01x05_Socket_2")
 		(lib_id "Connector:Conn_01x05_Socket")
 		(at 198.12 54.61 0)
@@
 	)
 	(symbol
+		(lib_id "Jumper:SolderJumper_2_Open")
+		(at 185.42 82.55 0)
+		(unit 1)
+		(exclude_from_sim no)
+		(in_bom no)
+		(on_board yes)
+		(dnp no)
+		(fields_autoplaced yes)
+		(property "Reference" "JP1002"
+			(at 185.42 76.2 0)
+			(effects
+				(font
+					(size 1.27 1.27)
+				)
+				(hide yes)
+			)
+		)
+		(property "Value" "SolderJumper_2_Open"
+			(at 185.42 78.74 0)
+			(effects
+				(font
+					(size 1.27 1.27)
+				)
+				(hide yes)
+			)
+		)
+		(property "Footprint" ""
+			(at 185.42 82.55 0)
+			(effects
+				(font
+					(size 1.27 1.27)
+				)
+				(hide yes)
+			)
+		)
+		(property "Datasheet" "~"
+			(at 185.42 82.55 0)
+			(effects
+				(font
+					(size 1.27 1.27)
+				)
+				(hide yes)
+			)
+		)
+		(property "Description" "Solder Jumper, 2-pole, open"
+			(at 185.42 82.55 0)
+			(effects
+				(font
+					(size 1.27 1.27)
+				)
+				(hide yes)
+			)
+		)
+		(pin "1"
+		)
+		(pin "2"
+		)
+		(instances
+			(project "testcircuit"
+				(path "/bd96de00-d7fe-4095-9be4-fc1fde628ce9"
+					(reference "JP1002")
+					(unit 1)
+				)
+			)
+		)
+	)
+	(symbol
 		(lib_id "power:GND")
 		(at 203.2 73.66 0)
@@
 	)
 	(symbol
+		(lib_name "Conn_01x05_Socket_1")
 		(lib_id "Connector:Conn_01x05_Socket")
 		(at 198.12 69.85 0)
@@
 				(path "/bd96de00-d7fe-4095-9be4-fc1fde628ce9"
 					(reference "J1003")
+					(unit 1)
+				)
+			)
+		)
+	)
+	(symbol
+		(lib_id "Jumper:SolderJumper_2_Open")
+		(at 185.42 80.01 0)
+		(unit 1)
+		(exclude_from_sim no)
+		(in_bom no)
+		(on_board yes)
+		(dnp no)
+		(fields_autoplaced yes)
+		(property "Reference" "JP1001"
+			(at 185.42 73.66 0)
+			(effects
+				(font
+					(size 1.27 1.27)
+				)
+				(hide yes)
+			)
+		)
+		(property "Value" "SolderJumper_2_Open"
+			(at 185.42 76.2 0)
+			(effects
+				(font
+					(size 1.27 1.27)
+				)
+				(hide yes)
+			)
+		)
+		(property "Footprint" ""
+			(at 185.42 80.01 0)
+			(effects
+				(font
+					(size 1.27 1.27)
+				)
+				(hide yes)
+			)
+		)
+		(property "Datasheet" "~"
+			(at 185.42 80.01 0)
+			(effects
+				(font
+					(size 1.27 1.27)
+				)
+				(hide yes)
+			)
+		)
+		(property "Description" "Solder Jumper, 2-pole, open"
+			(at 185.42 80.01 0)
+			(effects
+				(font
+					(size 1.27 1.27)
+				)
+				(hide yes)
+			)
+		)
+		(pin "1"
+		)
+		(pin "2"
+		)
+		(instances
+			(project ""
+				(path "/bd96de00-d7fe-4095-9be4-fc1fde628ce9"
+					(reference "JP1001")
 					(unit 1)
 				)
@@
 		(lib_id "Device:R_US")
 		(at 184.15 87.63 90)
+		(mirror x)
 		(unit 1)
 		(exclude_from_sim no)
@@
 		(on_board yes)
 		(dnp no)
-		(fields_autoplaced yes)
 		(property "Reference" "R1001"
-			(at 184.15 81.28 90)
+			(at 184.15 93.98 90)
 			(effects
 				(font
@@
 		)
 		(property "Value" "2K"
-			(at 184.15 83.82 90)
+			(at 184.15 91.44 90)
 			(effects
 				(font
@@
 		)
 		(property "Footprint" ""
-			(at 184.404 86.614 90)
-			(effects
-				(font
+			(at 184.404 88.646 90)
+			(effects
+				(font
